File: ESP8266_Water_Sensor/ESP8266_Water_Sensor.sch (KiCad schematic (older format))
At the start: 38 parts, among them J1 Conn_01x06_Female, J2 691137710002, J3 691137710003, J4 691137710002, J5 Conn_01x06_Female, U1 ESP-WROOM-02D_M1102H3200PH3Q0_, U2 AP6502SP-13

Commit message: edited the silkscreen
Parts:
- H1, H2: footprint MountingHole:MountingHole_3.2mm_M3 -> MountingHole:MountingHole_2.7mm_M2.5
Changed lines of the file:
@@
 F 0 "H2" H 10550 5996 50  0000 L CNN
 F 1 "MountingHole" H 10550 5905 50  0000 L CNN
-F 2 "MountingHole:MountingHole_3.2mm_M3" H 10450 5950 50  0001 C CNN
+F 2 "MountingHole:MountingHole_2.7mm_M2.5" H 10450 5950 50  0001 C CNN
 F 3 "~" H 10450 5950 50  0001 C CNN
 	1    10450 5950
@@
 F 0 "H1" H 10550 5796 50  0000 L CNN
 F 1 "MountingHole" H 10550 5705 50  0000 L CNN
-F 2 "MountingHole:MountingHole_3.2mm_M3" H 10450 5750 50  0001 C CNN
+F 2 "MountingHole:MountingHole_2.7mm_M2.5" H 10450 5750 50  0001 C CNN
 F 3 "~" H 10450 5750 50  0001 C CNN
 	1    10450 5750
