File: ESP32_12v_Relay/ESP32_12v_Relay.sch (KiCad schematic (older format))
At the start: 49 parts, among them IC1 DMN2029USD-13, IC2 DMN2029USD-13, J1 691137710002, J2 691137710002, J3 691137710002, J4 691137710002, J5 Conn_01x06_Female, J6 691137710002, U1 ESP32-C3-WROOM-02-H4, U2 AP6502SP-13

Commit message: Cleaned up projects
Parts:
- D5: renamed from D?; footprint (none) -> LED_SMD:LED_0805_2012Metric_Pad1.15x1.40mm_HandSolder
- F1: value 5A -> 7A
- gave numbers to parts that had none: 1
Changed lines of the file:
@@
 P 5200 7150
 F 0 "F1" V 5003 7150 50  0000 C CNN
-F 1 "5A" V 5094 7150 50  0000 C CNN
+F 1 "7A" V 5094 7150 50  0000 C CNN
 F 2 "Fuse:Fuse_1206_3216Metric_Pad1.42x1.75mm_HandSolder" V 5130 7150 50  0001 C CNN
 F 3 "~" H 5200 7150 50  0001 C CNN
@@
 $EndComp
 $Comp
-L Device:LED D?
+L Device:LED D5
 U 1 1 61711833
 P 2550 4200
-F 0 "D?" V 2589 4082 50  0000 R CNN
+F 0 "D5" V 2589 4082 50  0000 R CNN
 F 1 "LED" V 2498 4082 50  0000 R CNN
-F 2 "" H 2550 4200 50  0001 C CNN
+F 2 "LED_SMD:LED_0805_2012Metric_Pad1.15x1.40mm_HandSolder" H 2550 4200 50  0001 C CNN
 F 3 "~" H 2550 4200 50  0001 C CNN
 	1    2550 4200
@@
 $EndComp
 $Comp
-L Device:R R?
+L Device:R R13
 U 1 1 61713B87
 P 2550 3800
-F 0 "R?" H 2620 3846 50  0000 L CNN
+F 0 "R13" H 2620 3846 50  0000 L CNN
 F 1 "66.5" H 2620 3755 50  0000 L CNN
 F 2 "Resistor_SMD:R_0805_2012Metric_Pad1.20x1.40mm_HandSolder" V 2480 3800 50  0001 C CNN
@@
 $EndComp
 $Comp
-L power:+3V3 #PWR?
+L power:+3V3 #PWR033
 U 1 1 61714614
 P 2550 3550
-F 0 "#PWR?" H 2550 3400 50  0001 C CNN
+F 0 "#PWR033" H 2550 3400 50  0001 C CNN
 F 1 "+3V3" H 2565 3723 50  0000 C CNN
 F 2 "" H 2550 3550 50  0001 C CNN
@@
 $EndComp
 $Comp
-L power:GND #PWR?
+L power:GND #PWR036
 U 1 1 61714E83
 P 2550 4450
-F 0 "#PWR?" H 2550 4200 50  0001 C CNN
+F 0 "#PWR036" H 2550 4200 50  0001 C CNN
 F 1 "GND" H 2555 4277 50  0000 C CNN
 F 2 "" H 2550 4450 50  0001 C CNN
